File: kicad/FirstHCProject.kicad_pcb (KiCad board)
At the start: 2 copper layers, 61.7 x 74.6 mm, 17 parts, among them Q1 2N3904

Commit message: resubmit
Parts:
- added G***: LOGO, LOGO, B.Cu at (154.1, 127.6)
- added G***: LOGO, LOGO, B.Cu at (156.1, 89.6)
- added G***: LOGO, LOGO, B.Cu at (146.4, 108.4)
Other:
- board text added: "LED"
